File: kicad/beanport.kicad_sch (KiCad schematic)
At the start: 5 parts, among them U1 SN74LVC245APW, U2 SN74LVC245APW, U3 74LS138

Commit message: A0 => RS(A0)
Connections:
- net A0 3v3 renamed RS(A0) 3v3
Changed lines of the file:
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@@
 		)
 	)
-	(label "A0 3v3"
+	(label "RS(A0) 3v3"
 		(at 114.3 64.77 0)
 		(effects
